File: laser.brd (EAGLE design)
At the start: 74.9 x 82.5 mm, 19 parts

Commit message: Continue to route
Parts:
- removed NANO: NANO, jet-lib:PDIP-32
- removed X_AXIS_CON, Y_AXIS_CON: (no value), SparkFun-Connectors:1X04_LONGPADS
- added E$10, E$11, E$12, E$15, E$16: (no value), jumper:0R/10
- added E$13, E$14, E$3: (no value), pinhead:1X04
- added E$2: (no value), pinhead:1X03
- added E$5: (no value), pinhead:1X15
- moved E$9 4.02 mm to (49.5, 61.0)
Connections:
- new net S$23: E$10.1, END_Y.1
- new net S$24: E$11.1, END_X.1
- new net S$25: E$12.2, Y_AXIS.GND1, Y_AXIS.GND2
- new net S$26: E$15.1, E$16.2
- new net S$27: E$16.1, Y_AXIS.M+
- net 12V: now also E$15.2; no longer Y_AXIS.M+
- net 5V: now also E$3.4; no longer NANO.D9
- net GND: now also E$12.1, E$3.2, E$5.12; no longer NANO.A7, NANO.D11, Y_AXIS.GND1, Y_AXIS.GND2
- net S$1: now also E$5.10; no longer NANO.A5
- net S$10: now also E$14.1, Y_AXIS.A1; no longer X_AXIS.B1, X_AXIS_CON.1
- net S$11: now also E$13.4, X_AXIS.B1; no longer Y_AXIS.B1, Y_AXIS_CON.1
- net S$12: now also E$13.3, X_AXIS.B2; no longer Y_AXIS.B2, Y_AXIS_CON.2
- net S$13: now also E$13.2, X_AXIS.A2; no longer Y_AXIS.A2, Y_AXIS_CON.3
- net S$14: now also E$13.1, X_AXIS.A1; no longer Y_AXIS.A1, Y_AXIS_CON.4
- net S$15: now also E$11.2, E$5.4; no longer END_Y.1, NANO.+5V
- net S$17: now also E$10.2, E$5.3; no longer END_X.1, NANO.RESET1
- net S$2: now also E$5.11; no longer NANO.A6
- net S$3: now also E$5.8; no longer NANO.A3
- net S$4: now also E$5.7; no longer NANO.A2
- net S$6: now also E$5.2; no longer NANO.GND1
- net S$7: now also E$14.4, Y_AXIS.B1; no longer X_AXIS.A1, X_AXIS_CON.4
- net S$8: now also E$14.3, Y_AXIS.B2; no longer X_AXIS.A2, X_AXIS_CON.3
- net S$9: now also E$14.2, Y_AXIS.A2; no longer X_AXIS.B2, X_AXIS_CON.2
Routing:
- net GND: track 0.00 -> 241.7 mm
- net 12V: track 0.00 -> 151.5 mm
- net S$3: track 0.00 -> 140.4 mm
- net 5V: track 0.00 -> 121.4 mm
- net S$2: track 0.00 -> 96.2 mm
- net S$24: track 0.00 -> 57.1 mm
- net S$23: track 0.00 -> 56.8 mm
- net S$5: track 0.00 -> 55.8 mm
- net S$7: track 0.00 -> 50.7 mm
- net S$8: track 0.00 -> 48.9 mm
- net S$4: track 0.00 -> 48.4 mm
- net S$9: track 0.00 -> 47.1 mm
- net S$10: track 0.00 -> 45.3 mm
- net S$1: track 0.00 -> 41.6 mm
- net S$21: track 0.00 -> 31.3 mm
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- added copper zone on layer 16, net GND

Commit message: First version
Parts:
- removed FAN: (no value), pinhead:1X02
- added FAN2: (no value), pinhead:1X02
- E$4: value (none) -> 5Ω
- E$6: value (none) -> 50Ω
- E$8: value (none) -> 1N4001
- E$9: value (none) -> 220Ω
- moved FAN1 7.62 mm to (69.8, 20.3)
- moved E$9 1.27 mm to (50.8, 61.0)
- renumbered E$13 to X_MOTOR, E$14 to Y_MOTOR, E$7 to NPN
Connections:
- new net S$28: DC_JACK.GND@1, E$12.1
- net 12V: now also FAN2.2; no longer FAN.2
- net GND: now also FAN2.1; no longer DC_JACK.GND@1, E$12.1, FAN.1
Routing:
- net S$28: track 0.00 -> 38.5 mm
- net S$3: track 140.4 -> 147.3 mm
- net S$20: track 0.00 -> 4.97 mm
- net GND: track 241.7 -> 239.2 mm
- net S$6: track 12.5 -> 13.0 mm
- added copper zone on layer 16, net 5V
- added copper zone on layer 16, net S$25
- added copper zone on layer 16, net S$28
- added copper zone on layer 16, net S$29
- added copper zone on layer 16, net S$30
- added copper zone on layer 16, net S$31
- added copper zone on layer 16, net S$32
Other:
- board text added: "Aoshido"
- board text added: "Nano"
